Commit message: mesaures

File: tas_car_description/urdf/include/macros.xacro (robot description, xacro)
@@ -214,5 +214,5 @@
         <joint name="hokuyo_joint" type="fixed">
             <axis xyz="0 1 0" />
-            <origin xyz="${-laser_size+chassis_length/2} 0 ${laser_size+tire_radius + chassis_height/2}" rpy="0 0 0"/>
+            <origin xyz="${-laser_size+chassis_length/2} 0 ${tire_radius + 0.03}" rpy="0 0 0"/>
             <parent link="chassis"/>
             <child link="hokuyo_link"/>

File: tas_car_description/urdf/tas_car_description.urdf.xacro (robot description, xacro)
@@ -7,7 +7,7 @@
     <xacro:property name="PI"         value="3.1415926535897931" />
     <!-- Chassis. -->
-    <xacro:property name="chassis_length" value="0.358" />
-    <xacro:property name="chassis_width"  value="0.18" />
-    <xacro:property name="chassis_height" value="0.068" />
+    <xacro:property name="chassis_length" value="0.346" />
+    <xacro:property name="chassis_width"  value="0.17" />
+    <xacro:property name="chassis_height" value="0.095" />
     <xacro:property name="chassis_mass"   value="3" />
     <!-- hub_diameter and tire_diameter are the diameters of the hub and tire,
@@ -31,5 +31,5 @@
     <xacro:property name="axle_length" value="0.03"/>
     <xacro:property name="wheel_travel" value="0.084"/>
-    <xacro:property name="shock_z_offset" value="0.0655"/>
+    <xacro:property name="shock_z_offset" value="0.0055"/>
     <!-- TODO get shock sprint constant, default used here -->
     <!-- shock_eff_limit is 2 * ((shock_stroke / 2) * shock_spring_constant) N.

Commit message: automatization

File: tas_car_description/urdf/include/macros.xacro (robot description, xacro)
@@ -79,7 +79,4 @@
             </solid_cuboid_inertial>
         </link>
-        <gazebo reference="chassis">
-            <material>Gazebo/Orange</material>
-        </gazebo>
         <!-- Fix the chassis to the base_link. -->
         <joint name="base_link_to_chassis" type="fixed">
@@ -239,3 +236,15 @@
         </link>
     </macro>
+    <!-- IMU link. -->
+    <macro name="imu_link">
+        <link name="imu_link">
+            <null_inertial/>
+        </link>
+        <!-- Fix the imu_link to the chassis. -->
+        <joint name="imu_link_to_chassis" type="fixed">
+            <parent link="chassis"/>
+            <child link="imu_link"/>
+            <origin xyz="-0.28 0.0 0.15" rpy="0 0 0"/>
+        </joint>
+    </macro>
 </robot>

File: tas_car_description/urdf/tas_car_description.urdf.xacro (robot description, xacro)
@@ -1,5 +1,7 @@
 <?xml version="1.0"?>
 <!-- Description of the tas_car. -->
-<robot name="tas_car" xmlns:xacro="http://www.ros.org/wiki/xacro">
+<robot name="tas_car" xmlns:xacro="http://www.ros.org/wiki/xacro"
+    xmlns:controller="http://playerstage.sourceforge.net/gazebo/xmlschema/#controller"
+    xmlns:interface="http://playerstage.sourceforge.net/gazebo/xmlschema/#interface">
     <!-- Physical constants. -->
     <xacro:property name="degrees_45" value="0.785398163" />
@@ -95,6 +97,11 @@
     <!-- Laser scanner. -->
     <xacro:hokuyo_laser />
+    <!-- imu -->
+    <xacro:imu_link/>
     <gazebo>
         <plugin name="gazebo_ros_control" filename="libgazebo_ros_control.so"/>
     </gazebo>
+    <gazebo reference="chassis">
+      <material>Gazebo/Orange</material>
+    </gazebo>
 </robot>
